Commit message: implemented car description for carrellino

File: src/0_sensors/car_description/src/urdf/materials.urdf.xacro (robot description, xacro)
@@ -16,3 +16,6 @@
         <color rgba="0.8 0.0 0.0 1.0"/>
     </material>
+    <material name="Green">
+        <color rgba="0.0 0.8 0.0 1.0"/>
+    </material>
 </robot>

File: src/0_sensors/car_description/src/urdf/sensors/imu.urdf.xacro (robot description, xacro)
@@ -4,5 +4,5 @@
         <link name="${name}_link">
             <visual name="">
-                <origin xyz="0.0 0.0 0.0" rpy="0.0 0.0 0.0"/>
+                <origin xyz="0.1 0.0 0.0" rpy="0.0 0.0 0.0"/>
                 <geometry>
                     <box size="0.05 0.05 0.02"/>
@@ -13,5 +13,5 @@
         <link name="vehicle">
             <visual name="">
-                <origin xyz="-1.6 0.0 0.0" rpy="0.0 0.0 0.0"/>
+                <origin xyz="0 0.0 0.0" rpy="0.0 0.0 0.0"/>
                 <geometry>
                     <box size="0.05 0.05 0.02"/>
@@ -20,5 +20,5 @@
         </link>
         <joint name="${name}_base_joint" type="fixed">
-            <origin xyz="-1.6 0.0 0.0" rpy="0.0 0.0 0.0"/>
+            <origin xyz="0.1 0.0 0.0" rpy="0.0 0.0 0.0"/>
             <xacro:insert_block name="origin"/>
             <parent link="${name}_link"/>
